Commit message: QP controller for the arm IK and control [wip]

File: upperBody_description/upperBody.xacro (robot description, xacro)
@@ -3,6 +3,6 @@
 	<!-- These values must be entered manually -->
 	<!-- Average BMI = 22. If above, enter 1, else enter 0 -->
-	<xacro:property name="bodyHeight" value="1.83" />
-	<xacro:property name="bodyMass" value="88" />
+	<xacro:property name="bodyHeight" value="1.80" />
+	<xacro:property name="bodyMass" value="110" />
 	<xacro:property name="BMI" value="${bodyMass/(bodyHeight*bodyHeight)}" />
 	<xacro:property name="isBMIgreaterThanAverage" value="0"/>
@@ -145,5 +145,5 @@
 				<box size="${pelvis_depth} ${pelvis_width} ${pelvis_length}"/>
 			</geometry>
-			<origin rpy="0 0 0" xyz="0 0 ${pelvis_length/2-hip_thickness}"/>
+			<origin rpy="0 0 0" xyz="0 0 ${pelvis_length/2}"/>
 			<material name="blue" />
 		</visual>
@@ -152,9 +152,9 @@
 				<box size="${collision_depth_factor*pelvis_depth} ${collision_width_factor*pelvis_width} ${collision_height_factor*pelvis_length}"/>
 			</geometry>
-			<origin rpy="0 0 0" xyz="0 0 ${pelvis_length/2-hip_thickness}"/>
+			<origin rpy="0 0 0" xyz="0 0 ${pelvis_length/2}"/>
 		</collision>
 		<inertial>
 			<mass value="${0.7*pelvis_mass}" />
-			<origin rpy="0 0 0" xyz="0 0 ${pelvis_length/2-hip_thickness}"/>
+			<origin rpy="0 0 0" xyz="0 0 ${pelvis_length/2}"/>
 			<xacro:box_inertia m="${0.7*pelvis_mass}" Lx="${pelvis_depth}" Ly="${pelvis_width}" Lz="${pelvis_length}"/>
 		</inertial>
@@ -283,18 +283,4 @@
 		</inertial>
 	</link>
-<joint name="right_hand_fixed" type="fixed">
-   <origin rpy="0 0 0 " xyz="0.0 0.0 ${hand_length / 2}"/>
-   <child link="right_hand_gripper"/>
-   <parent link="right_hand"/>
-   <axis use_parent_model_frame="1" xyz="0 0 0"/>
-   <dynamics damping="0" friction="0" spring_reference="0" spring_stiffness="0"/>
- </joint>
- <link name="right_hand_gripper">
-   <inertial>
-     <origin xyz="0 0 0"/>
-     <mass value="0.000001"/>
-     <inertia ixx="0.000001" ixy="0.000001" ixz="0.000001" iyy="0.000001" iyz="0.000001" izz="0.000001"/>
-   </inertial>
- </link>
 <xacro:virtual_body name="body_T4_left_clavicular" m="${0.1*thoracicspine_mass}"/>
 <link name="left_clavicular">
@@ -378,5 +364,5 @@
 	<!-- Define joints -->
 	<!-- Back joints -->
-	<joint name="lumbarspine_X" type="revolute">
+	<joint name="lumbarspine_X" type="fixed">
 		<parent link="pelvis"/>
 		<child link="body_L5_1"/>
@@ -387,5 +373,5 @@
 		<dynamics damping="${jointDamping}" friction="${jointFriction}"/>
 	</joint>
-	<joint name="lumbarspine_Y" type="revolute">
+	<joint name="lumbarspine_Y" type="fixed">
 		<parent link="body_L5_1"/>
 		<child link="body_L5_2"/>
@@ -396,5 +382,5 @@
 		<dynamics damping="${jointDamping}" friction="${jointFriction}"/>
 	</joint>
-	<joint name="lumbarspine_Z" type="revolute">
+	<joint name="lumbarspine_Z" type="fixed">
 		<parent link="body_L5_2"/>
 		<child link="lumbar_spine"/>
@@ -404,5 +390,5 @@
 		<dynamics damping="${jointDamping}" friction="${jointFriction}"/>
 	</joint>
-	<joint name="thoracicspine_X" type="revolute">
+	<joint name="thoracicspine_X" type="fixed">
 		<parent link="lumbar_spine"/>
 		<child link="body_T8_1"/>
@@ -412,5 +398,5 @@
 		<dynamics damping="${jointDamping}" friction="${jointFriction}"/>
 	</joint>
-	<joint name="thoracicspine_Y" type="revolute">
+	<joint name="thoracicspine_Y" type="fixed">
 		<parent link="body_T8_1"/>
 		<child link="body_T8_2"/>
@@ -420,5 +406,5 @@
 		<dynamics damping="${jointDamping}" friction="${jointFriction}"/>
 	</joint>
-	<joint name="thoracicspine_Z" type="revolute">
+	<joint name="thoracicspine_Z" type="fixed">
 		<parent link="body_T8_2"/>
 		<child link="thoracic_spine"/>
@@ -429,5 +415,5 @@
 	</joint>
 	<!-- Right arm joints -->
-	<joint name="right_clavicular_X" type="revolute">
+	<joint name="right_clavicular_X" type="fixed">
     <!-- flexion (elevation) -->
 		<parent link="thoracic_spine"/>
@@ -438,5 +424,5 @@
 		<dynamics damping="${jointDamping}" friction="${jointFriction}"/>
 	</joint>
-	<joint name="right_clavicular_Y" type="revolute">
+	<joint name="right_clavicular_Y" type="fixed">
     <!-- abduction -->
 		<parent link="body_T4_right_clavicular"/>
@@ -453,5 +439,5 @@
 		<axis xyz="1 0 0"/>
 		<origin xyz="0 0 ${CSJ_shoulder}"/>
-		<limit effort="${69*forceCapacity}" lower="-1.571" upper="${PI}" velocity="${maxVelJoint}"/>
+		<limit effort="${69*forceCapacity}" lower="0" upper="${PI}" velocity="${maxVelJoint}"/>
 		<dynamics damping="${jointDamping}" friction="${jointFriction}"/>
 	</joint>
@@ -462,5 +448,5 @@
 		<axis xyz="0 1 0"/>
 		<origin xyz="0 0 0"/>
-		<limit effort="${90*forceCapacity}" lower="${-PI/2}" upper="${PI/2}" velocity="${maxVelJoint}"/>
+		<limit effort="${90*forceCapacity}" lower="${0}" upper="${PI/4}" velocity="${maxVelJoint}"/>
 		<dynamics damping="${jointDamping}" friction="${jointFriction}"/>
 	</joint>
@@ -471,5 +457,5 @@
 		<axis xyz="0 0 1"/>
 		<origin xyz="0 0 0"/>
-		<limit effort="${51*forceCapacity}" lower="-1.658" upper="1.396" velocity="${maxVelJoint}"/>
+		<limit effort="${51*forceCapacity}" lower="0" upper="${PI/2}" velocity="${maxVelJoint}"/>
 		<dynamics damping="${jointDamping}" friction="${jointFriction}"/>
 	</joint>
@@ -484,5 +470,5 @@
 		<dynamics damping="${jointDamping}" friction="${jointFriction}"/>
 	</joint>
-	<joint name="right_elbow_Z" type="revolute">
+	<joint name="right_elbow_Z" type="fixed">
     <!-- pronosupination -->
 		<parent link="body_right_elbow"/>
@@ -493,5 +479,5 @@
 		<dynamics damping="${jointDamping}" friction="${jointFriction}"/>
 	</joint>
-	<joint name="right_wrist_X" type="revolute">
+	<joint name="right_wrist_X" type="fixed">
     <!-- flexion -->
 		<parent link="right_forearm"/>
@@ -502,5 +488,5 @@
 		<dynamics damping="${jointDamping}" friction="${jointFriction}"/>
 	</joint>
-	<joint name="right_wrist_Y" type="revolute">
+	<joint name="right_wrist_Y" type="fixed">
     <!-- abduction -->
 		<parent link="body_right_wrist"/>
@@ -511,5 +497,5 @@
 		<dynamics damping="${jointDamping}" friction="${jointFriction}"/>
 	</joint>
-	<joint name="left_clavicular_X" type="revolute">
+	<joint name="left_clavicular_X" type="fixed">
     <!-- flexion (elevation) -->
 		<parent link="thoracic_spine"/>
@@ -521,5 +507,5 @@
 		<dynamics damping="${jointDamping}" friction="${jointFriction}"/>
 	</joint>
-	<joint name="left_clavicular_Y" type="revolute">
+	<joint name="left_clavicular_Y" type="fixed">
     <!-- abduction -->
 		<parent link="body_T4_left_clavicular"/>
@@ -531,5 +517,5 @@
 		<dynamics damping="${jointDamping}" friction="${jointFriction}"/>
 	</joint>
-	<joint name="left_shoulder_X" type="revolute">
+	<joint name="left_shoulder_X" type="fixed">
     <!-- abduction -->
 		<parent link="left_clavicular"/>
@@ -540,5 +526,5 @@
 		<dynamics damping="${jointDamping}" friction="${jointFriction}"/>
 	</joint>
-	<joint name="left_shoulder_Y" type="revolute">
+	<joint name="left_shoulder_Y" type="fixed">
     <!-- flexion -->
 		<parent link="body_left_shoulder_1"/>
@@ -549,5 +535,5 @@
 		<dynamics damping="${jointDamping}" friction="${jointFriction}"/>
 	</joint>
-	<joint name="left_shoulder_Z" type="revolute">
+	<joint name="left_shoulder_Z" type="fixed">
     <!-- rotation -->
 		<parent link="body_left_shoulder_2"/>
@@ -558,5 +544,5 @@
 		<dynamics damping="${jointDamping}" friction="${jointFriction}"/>
 	</joint>
-	<joint name="left_elbow_Y" type="revolute">
+	<joint name="left_elbow_Y" type="fixed">
     <!-- flexion -->
 		<parent link="left_arm"/>
@@ -568,5 +554,5 @@
 		<dynamics damping="${jointDamping}" friction="${jointFriction}"/>
 	</joint>
-	<joint name="left_elbow_Z" type="revolute">
+	<joint name="left_elbow_Z" type="fixed">
     <!-- pronosupination -->
 		<parent link="body_left_elbow"/>
@@ -577,5 +563,5 @@
 		<dynamics damping="${jointDamping}" friction="${jointFriction}"/>
 	</joint>
-	<joint name="left_wrist_X" type="revolute">
+	<joint name="left_wrist_X" type="fixed">
     <!-- flexion -->
 		<parent link="left_forearm"/>
@@ -586,5 +572,5 @@
 		<dynamics damping="${jointDamping}" friction="${jointFriction}"/>
 	</joint>
-	<joint name="left_wrist_Y" type="revolute">
+	<joint name="left_wrist_Y" type="fixed">
     <!-- abduction -->
 		<parent link="body_left_wrist"/>
